File: hardware/atmos-fc/atmos-fc_power.kicad_sch (KiCad schematic)
At the start: 17 parts, among them U1 MAX25232, U2 TPS78533BQDRBRQ1

Commit message: Initial commit
Other:
- note added: "Max. Battery 8S"
- note removed: "+14V < BATT < +26V"
Changed lines of the file:
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@@
 		)
 	)
-	(text "+14V < BATT < +26V"
+	(text "Max. Battery 8S"
 		(exclude_from_sim no)
-		(at 37.846 71.12 0)
+		(at 35.56 72.644 0)
 		(effects
 			(font

Commit message: Add GYRO_1_EXTI Pin
Other:
- note added: "Max. Battery 6S"
- note removed: "Max. Battery 8S"
Changed lines of the file:
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@@
 		)
 	)
-	(text "Max. Battery 8S"
+	(text "Max. Battery 6S"
 		(exclude_from_sim no)
 		(at 35.56 72.644 0)
